File: interface_MTM800E_V4.kicad_pcb (KiCad board)
At the start: 2 copper layers, 85.2 x 55.4 mm, 72 parts, among them J1 Raspberry_Pi_2_3, J10 Conn_01x01, J11 Conn_01x01, J12 Screw_Terminal_01x02, J13 Screw_Terminal_01x02, J14 Conn_01x02, J15 Screw_Terminal_01x02, J16 Conn_01x01, J2 Conn_01x01_Male, J3 Conn_02x10_Odd_Even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

Commit message: V4.0-a
Parts:
- removed H1: MountingHole_Pad, Connector_Wire:SolderWirePad_1x01_Drill0.8mm
- added J17: Conn_01x01_Male, Connector_PinHeader_2.54mm:PinHeader_1x01_P2.54mm_Vertical, F.Cu at (127.3, 92.5)
Connections:
- net /EXT_PTT renamed EXT_PTT
- net /PTT renamed CMD_PTT
Routing:
- net Hp_Son: track 40.8 -> 41.4 mm

Commit message: v4b
Parts:
- removed J7: Conn_02x06_Odd_Even, Connector_PinHeader_2.54mm:PinHeader_2x06_P2.54mm_Vertical
- added J7‎: Conn_02x07_Odd_Even, Connector_PinHeader_2.54mm:PinHeader_2x07_P2.54mm_Vertical, F.Cu at (126.2, 76.7)
- J6: value Conn_02x06_Odd_Even -> Conn_02x07_Odd_Even; footprint Connector_PinHeader_2.54mm:PinHeader_2x06_P2.54mm_Vertical -> Connector_PinHeader_2.54mm:PinHeader_2x07_P2.54mm_Vertical
- moved J17 12.6 mm to (116.7, 99.3)
- moved J6 2.54 mm to (126.2, 57.4)
Connections:
- J6 pad 10: /UART1RXD -> /SCITXD
- J6 pad 12: /UART2RXD -> /UART1RXD
- J6 pad 2: /SCITXD -> /RXDMax
- J6 pad 4: /UART1RXD -> /SCITXD
- J6 pad 6: /UART2RXD -> /UART1RXD
- J6 pad 7: /TXDMax -> /TxDPi
- J6 pad 8: /SCITXD -> /UART2RXD
Routing:
- net /RXDMax: track 77.0 -> 101.4 mm, vias 0 -> 1
- net /UART1RTS: track 29.9 -> 12.0 mm
- net /UART1RXD: track 59.8 -> 72.2 mm, vias 4 -> 5
- net /UART2RXD: track 28.6 -> 35.9 mm
- net /UART1TXD: track 49.7 -> 56.9 mm
- net /RxDPi: track 28.4 -> 33.6 mm
- net /SCITXD: track 69.1 -> 73.4 mm
- net /SCIRXD: track 50.2 -> 46.1 mm
- net /TXDMax: track 82.1 -> 78.2 mm
- net /UART2TXD: track 28.8 -> 31.4 mm
- net /TxDPi: track 12.3 -> 14.1 mm
