File: interface_MTM800E_V4.kicad_pcb (KiCad board)
At the start: 2 copper layers, 85.2 x 55.4 mm, 72 parts, among them J1 Raspberry_Pi_2_3, J10 Conn_01x01, J11 Conn_01x01, J12 Screw_Terminal_01x02, J13 Screw_Terminal_01x02, J14 Conn_01x02, J15 Screw_Terminal_01x02, J16 Conn_01x01, J17 Conn_01x01_Male, J2 Conn_01x01_Male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

Commit message: v4f
Parts:
- R10, R8: footprint Resistor_THT:R_Axial_DIN0204_L3.6mm_D1.6mm_P2.54mm_Vertical -> Resistor_THT:R_Axial_DIN0207_L6.3mm_D2.5mm_P7.62mm_Horizontal
- R9: footprint Resistor_THT:R_Axial_DIN0207_L6.3mm_D2.5mm_P2.54mm_Vertical -> Resistor_THT:R_Axial_DIN0204_L3.6mm_D1.6mm_P2.54mm_Vertical
- moved R9 1.97 mm to (93.3, 93.8)
- moved R10 0.57 mm to (87.1, 101.7)
- moved R8 0.06 mm to (87.1, 98.7)
Routing:
- net /RXDMax: track 101.5 -> 97.1 mm
- net +3V3: track 69.5 -> 72.0 mm
- net /EXTMICAUD: track 48.8 -> 50.1 mm
- net /TXDMax: track 77.4 -> 76.6 mm
- net Net-(D2-Pad2): track 3.77 -> 3.01 mm
- net GND: track 93.2 -> 93.9 mm
- net Net-(R9-Pad1): track 3.46 -> 4.02 mm
Other:
- board text added: "Ignition"
