File: interface_MTM800E_V4.kicad_pcb (KiCad board)
At the start: 2 copper layers, 85.2 x 55.4 mm, 72 parts, among them J1 Raspberry_Pi_2_3, J10 Conn_01x01, J11 Conn_01x01, J12 Screw_Terminal_01x02, J13 Screw_Terminal_01x02, J14 Conn_01x02, J15 Screw_Terminal_01x02, J16 Conn_01x01, J17 Conn_01x01_Male, J2 Conn_01x01_Male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

Commit message: V4.1
Parts:
- added C18: 47µF, Capacitor_THT:CP_Radial_D4.0mm_P2.00mm, F.Cu at (83.6, 45.1)
- C8, C9: value 1µF -> 47µF
- R16: value 600 -> 680
- RV1, RV2: value 47k -> 1k
- moved J15 1.59 mm to (70.5, 99.6)
- moved C8 0.20 mm to (98.7, 62.9)
Connections:
- C8 pad 1: Net-(C8-Pad1) -> Hp_Son
- C8 pad 2: Hp_Son -> Net-(C8-Pad2)
- J1 pad 6: Net-(J1-Pad6) -> GND
- RV1 pad 1: Net-(C8-Pad1) -> Net-(C8-Pad2)
- RV2 pad 2: /RxAud -> Net-(C18-Pad1)
Routing:
- net GND: track 93.9 -> 91.7 mm
- net Hp_Son: track 41.4 -> 40.7 mm
Other:
- board text added: "TetraLink Svxlink V4.1-MTM F1IWQ Mars 2021"
- board text removed: "TetraLink Svxlink V4-MTM F1IWQ Mars 2021"

Commit message: V4.1
Parts:
- moved C18 24.4 mm to (68.8, 64.5)
- moved C17 5.11 mm to (64.0, 67.7)
- moved C15 2.11 mm to (62.7, 71.2)
Connections:
- J2 pad 2: /RxAud -> Net-(C18-Pad1)
- RV1 pad 1: Net-(C8-Pad2) -> Hp_Son
Routing:
- net Net-(C18-Pad1): track 0.00 -> 15.5 mm
- net GND: track 91.7 -> 105.6 mm
- net Hp_Son: track 40.7 -> 54.2 mm
- net Net-(C8-Pad1): track 5.49 -> 0.00 mm
- net /RxAud: track 4.99 -> 0.00 mm
- net Net-(RV4-Pad2): track 22.2 -> 20.4 mm
- net Net-(C15-Pad1): track 36.1 -> 34.6 mm
- net Net-(C15-Pad2): track 30.0 -> 31.1 mm
- net Net-(C17-Pad1): track 6.22 -> 7.22 mm
- net Net-(RV6-Pad2): track 32.1 -> 32.6 mm
Other:
- board text added: "TetraLink Svxlink V4.1-MTM F1IWQ Mars 2022"
- board text removed: "TetraLink Svxlink V4.1-MTM F1IWQ Mars 2021"
