File: interface_MTM800E_V4.sch (KiCad schematic (older format))
At the start: 46 parts, among them J1 Raspberry_Pi_2_3, J10 Conn_01x01, J11 Conn_01x01, J12 Screw_Terminal_01x02, J13 Screw_Terminal_01x02, J14 Conn_01x02, J16 Conn_01x01, J2 Conn_01x01_Male, J3 Conn_02x10_Odd_Even, J4 Conn_01x03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

Commit message: V4.0-a
Parts:
- removed D2: LED, LED_THT:LED_D3.0mm, symbol Device:LED
- removed H1: MountingHole_Pad, Connector_Wire:SolderWirePad_1x01_Drill0.8mm, symbol Mechanical:MountingHole_Pad
- removed J14: Conn_01x02, Connector_PinHeader_2.54mm:PinHeader_1x02_P2.54mm_Vertical, symbol Connector_Generic:Conn_01x02
- removed Q1: BC548, Package_TO_SOT_THT:TO-92_Inline_Wide, symbol Transistor_BJT:BC548
- removed R14: 100k, Resistor_THT:R_Axial_DIN0204_L3.6mm_D1.6mm_P2.54mm_Vertical, symbol Device:R
- removed R15: 100k, Resistor_THT:R_Axial_DIN0207_L6.3mm_D2.5mm_P7.62mm_Horizontal, symbol Device:R
- removed R5: 10k, Resistor_THT:R_Axial_DIN0207_L6.3mm_D2.5mm_P7.62mm_Horizontal, symbol Device:R
- removed R6: 330, Resistor_THT:R_Axial_DIN0207_L6.3mm_D2.5mm_P7.62mm_Horizontal, symbol Device:R
- added J17: Conn_01x01_Male, Connector_PinHeader_2.54mm:PinHeader_1x01_P2.54mm_Vertical, symbol Connector:Conn_01x01_Male
Connections:
- net labels added: CMD_PTT
- net labels removed: PTT
- wire segments 263 -> 245
Other:
- note added: "Connecteur MTM5x00"
- note removed: "Connecteur MTM5400"
- note removed: "J14 : \nsans/avec PTT"
- note removed: "PTT"
- moved on the sheet: C1, C2, D1, J13, J16, R18, R4, U3

Commit message: v4b
Parts:
- removed J6, J7: Conn_02x06_Odd_Even, Connector_PinHeader_2.54mm:PinHeader_2x06_P2.54mm_Vertical, symbol Connector_Generic:Conn_02x06_Odd_Even
- added J6, J7: Conn_02x07_Odd_Even, Connector_PinHeader_2.54mm:PinHeader_2x07_P2.54mm_Vertical, symbol Connector_Generic:Conn_02x07_Odd_Even
Connections:
- wire segments 245 -> 248
Other:
- note added: "3,3V"
- note added: "Audio vers MTM"
- note added: "MTM5x00 3,3V??"
- note added: "MTM800E 3,3V"
- note added: "entrée squelch\n radio si il doit \n être câblé"
- note removed: "Squelch repris depuis\npin 8 du TDA en interne\ndu MTM800E"
- moved on the sheet: C8, RV1
