File: interface_MTM800E_V4.sch (KiCad schematic (older format))
At the start: 39 parts, among them J1 Raspberry_Pi_2_3, J10 Conn_01x01, J11 Conn_01x01, J12 Screw_Terminal_01x02, J13 Screw_Terminal_01x02, J16 Conn_01x01, J17 Conn_01x01_Male, J2 Conn_01x01_Male, J3 Conn_02x10_Odd_Even, J4 Conn_01x03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

Commit message: v4f
Parts:
- R10, R8: footprint Resistor_THT:R_Axial_DIN0204_L3.6mm_D1.6mm_P2.54mm_Vertical -> Resistor_THT:R_Axial_DIN0207_L6.3mm_D2.5mm_P7.62mm_Horizontal
- R9: footprint Resistor_THT:R_Axial_DIN0207_L6.3mm_D2.5mm_P2.54mm_Vertical -> Resistor_THT:R_Axial_DIN0204_L3.6mm_D1.6mm_P2.54mm_Vertical
Connections:
- wire segments 248 -> 262
Other:
- note added: "DB9 J5"
- note added: "MTM5x00 3,3V"
- note removed: "MTM5x00 3,3V??"
Changed lines of the file:
@@
 F 0 "R9" V 1850 6850 50  0000 C CNN
 F 1 "1k" V 1850 6650 50  0000 C CNN
-F 2 "Resistor_THT:R_Axial_DIN0207_L6.3mm_D2.5mm_P2.54mm_Vertical" V 1880 6750 50  0001 C CNN
+F 2 "Resistor_THT:R_Axial_DIN0204_L3.6mm_D1.6mm_P2.54mm_Vertical" V 1880 6750 50  0001 C CNN
 F 3 "~" H 1950 6750 50  0001 C CNN
 	1    1950 6750
@@
 F 0 "R8" V 1850 6400 50  0000 L CNN
 F 1 "1k" V 1850 6200 50  0000 L CNN
-F 2 "Resistor_THT:R_Axial_DIN0204_L3.6mm_D1.6mm_P2.54mm_Vertical" V 1880 6350 50  0001 C CNN
+F 2 "Resistor_THT:R_Axial_DIN0207_L6.3mm_D2.5mm_P7.62mm_Horizontal" V 1880 6350 50  0001 C CNN
 F 3 "~" H 1950 6350 50  0001 C CNN
 	1    1950 6350
@@
 	2500 6550 2650 6550
 $Comp
-L Device:R R10
-U 1 1 5F495FED
-P 2250 6000
-F 0 "R10" H 2400 6050 50  0000 C CNN
-F 1 "10k" H 2400 5950 50  0000 C CNN
-F 2 "Resistor_THT:R_Axial_DIN0204_L3.6mm_D1.6mm_P2.54mm_Vertical" V 2180 6000 50  0001 C CNN
-F 3 "~" H 2250 6000 50  0001 C CNN
-	1    2250 6000
-	-1   0    0    1
-$EndComp
-$Comp
 L Device:R R11
 U 1 1 5F477AA4
@@
 	7800 2050 7800 2450
 Wire Wire Line
-	6050 3800 5500 3800
-Wire Wire Line
-	6050 4100 5500 4100
-Wire Wire Line
-	6050 4800 5500 4800
+	6050 3800 5950 3800
+Wire Wire Line
+	6050 4100 5950 4100
+Wire Wire Line
+	6050 4800 5950 4800
 Text Label 5500 3800 0    39   ~ 0
 TxDPi
@@
 MTM800E 3,3V
 Text Notes 7550 3950 0    35   ~ 0
-MTM5x00 3,3V??
+MTM5x00 3,3V
 Wire Notes Line
 	5300 3250 8050 3250
@@
 MTM800E 3,3V
 Text Notes 7550 4950 0    35   ~ 0
-MTM5x00 3,3V??
+MTM5x00 3,3V
 Text Notes 7500 4000 2    39   ~ 0
 -->
@@
 $EndComp
 Wire Wire Line
-	6050 4000 6050 3900
-Connection ~ 6050 3800
-Wire Wire Line
-	6050 3800 6050 3700
-Connection ~ 6050 3900
-Wire Wire Line
-	6050 3900 6050 3800
-Wire Wire Line
 	6550 3700 7350 3700
 Text Label 7000 3700 0    39   ~ 0
@@
 $EndComp
 Wire Wire Line
-	6050 5100 5500 5100
-Wire Wire Line
-	6050 5000 6050 4900
-Connection ~ 6050 4800
-Wire Wire Line
-	6050 4800 6050 4700
-Connection ~ 6050 4900
-Wire Wire Line
-	6050 4900 6050 4800
-Wire Wire Line
-	6050 5300 6050 5200
-Connection ~ 6050 5100
-Connection ~ 6050 5200
-Wire Wire Line
-	6050 5200 6050 5100
-Wire Wire Line
-	6050 4300 6050 4200
-Connection ~ 6050 4100
-Connection ~ 6050 4200
-Wire Wire Line
-	6050 4200 6050 4100
+	6050 5100 5950 5100
 Wire Wire Line
 	6550 4700 7350 4700
@@
 Wire Notes Line
 	8050 3250 8050 5450
+Text Notes 7550 3700 0    35   ~ 0
+DB9 J5
+Text Notes 7550 4700 0    35   ~ 0
+DB9 J5
+Wire Wire Line
+	6050 4000 5950 4000
+Wire Wire Line
+	5950 4000 5950 3900
+Wire Wire Line
+	5950 3700 6050 3700
+Wire Wire Line
+	6050 3900 5950 3900
+Connection ~ 5950 3900
+Wire Wire Line
+	5950 3900 5950 3800
+Connection ~ 5950 3800
+Wire Wire Line
+	5950 3800 5500 3800
+Wire Wire Line
+	5950 3800 5950 3700
+Wire Wire Line
+	6050 5000 5950 5000
+Wire Wire Line
+	5950 5000 5950 4900
+Connection ~ 5950 4800
+Wire Wire Line
+	5950 4800 5500 4800
+Wire Wire Line
+	6050 4900 5950 4900
+Connection ~ 5950 4900
+Wire Wire Line
+	5950 4900 5950 4800
+Wire Wire Line
+	5950 4800 5950 4700
+Wire Wire Line
+	5950 4700 6050 4700
+Wire Wire Line
+	5950 5100 5950 5200
+Wire Wire Line
+	5950 5300 6050 5300
+Connection ~ 5950 5100
+Wire Wire Line
+	5950 5100 5500 5100
+Wire Wire Line
+	6050 5200 5950 5200
+Connection ~ 5950 5200
+Wire Wire Line
+	5950 5200 5950 5300
+Wire Wire Line
+	6050 4300 5950 4300
+Wire Wire Line
+	5950 4300 5950 4200
+Connection ~ 5950 4100
+Wire Wire Line
+	5950 4100 5500 4100
+Wire Wire Line
+	5950 4200 6050 4200
+Connection ~ 5950 4200
+Wire Wire Line
+	5950 4200 5950 4100
+$Comp
+L Device:R R10
+U 1 1 5F495FED
+P 2250 6000
+F 0 "R10" H 2400 6050 50  0000 C CNN
+F 1 "10k" H 2400 5950 50  0000 C CNN
+F 2 "Resistor_THT:R_Axial_DIN0207_L6.3mm_D2.5mm_P7.62mm_Horizontal" V 2180 6000 50  0001 C CNN
+F 3 "~" H 2250 6000 50  0001 C CNN
+	1    2250 6000
+	-1   0    0    1
+$EndComp
 $EndSCHEMATC

Commit message: V4.1
Parts:
- added C18: 47µF, Capacitor_THT:CP_Radial_D4.0mm_P2.00mm, symbol Device:CP
- C8, C9: value 1µF -> 47µF
- RV1, RV2: value 47k -> 1k
Connections:
- wire segments 262 -> 265
- no-connect marks 47 -> 46
Other:
- note added: "cond 47µF"
Changed lines of the file:
@@
 encoding utf-8
 Sheet 1 2
-Title "Interface Raspberry V4 - MTM800(E) MTM5x00 pour SVXLink"
-Date "20/03/2021"
-Rev "4"
+Title "Interface Raspberry V4.1 - MTM800(E) MTM5x00 pour SVXLink"
+Date "20/01/2022"
+Rev "4.1"
 Comp "F1IWQ"
-Comment1 ""
+Comment1 "V4.1: chgt C8 - C9 : 47µF / Ajout C18 / RV1 RV2 : 10k"
 Comment2 ""
 Comment3 ""
@@
 P 6550 1750
 F 0 "RV1" H 6481 1796 50  0000 R CNN
-F 1 "47k" H 6481 1705 50  0000 R CNN
+F 1 "1k" H 6481 1705 50  0000 R CNN
 F 2 "Potentiometer_THT:Potentiometer_Bourns_3296W_Vertical" H 6550 1750 50  0001 C CNN
 F 3 "~" H 6550 1750 50  0001 C CNN
@@
 Wire Wire Line
 	2100 3600 2400 3600
-NoConn ~ 1700 3500
 NoConn ~ 1900 3500
 NoConn ~ 2000 3500
@@
 U 1 1 5EFD0977
 P 6350 1500
-F 0 "C8" V 6200 1350 50  0000 L CNN
-F 1 "1µF" V 6200 1550 50  0000 L CNN
+F 0 "C8" V 6550 1350 50  0000 L CNN
+F 1 "47µF" V 6450 1250 50  0000 L CNN
 F 2 "Capacitor_THT:CP_Radial_D4.0mm_P2.00mm" H 6388 1350 50  0001 C CNN
 F 3 "~" H 6350 1500 50  0001 C CNN
 	1    6350 1500
-	0    1    1    0
+	0    -1   -1   0
 $EndComp
 $Comp
@@
 P 7100 2500
 F 0 "C9" V 7250 2550 50  0000 L CNN
-F 1 "1µF" V 7250 2350 50  0000 L CNN
+F 1 "47µF" V 7250 2350 50  0000 L CNN
 F 2 "Capacitor_THT:CP_Radial_D4.0mm_P2.00mm" H 7138 2350 50  0001 C CNN
 F 3 "~" H 7100 2500 50  0001 C CNN
@@
 P 6550 2700
 F 0 "RV2" H 6480 2654 50  0000 R CNN
-F 1 "47k" H 6480 2745 50  0000 R CNN
+F 1 "1k" H 6480 2745 50  0000 R CNN
 F 2 "Potentiometer_THT:Potentiometer_Bourns_3296W_Vertical" H 6550 2700 50  0001 C CNN
 F 3 "~" H 6550 2700 50  0001 C CNN
@@
 $EndComp
 Wire Wire Line
-	6400 2700 5600 2700
+	6400 2700 6050 2700
 Text GLabel 4650 1300 0    39   Input ~ 0
 Squelch
@@
 	-1   0    0    1
 $EndComp
+Text Notes 7050 700  0    47   ~ 0
+cond 47µF
+Wire Wire Line
+	1800 3600 1700 3600
+Wire Wire Line
+	1700 3600 1700 3500
+$Comp
+L Device:CP C18
+U 1 1 61EC2114
+P 5900 2700
+F 0 "C18" V 6050 2750 50  0000 L CNN
+F 1 "47µF" V 6050 2550 50  0000 L CNN
+F 2 "Capacitor_THT:CP_Radial_D4.0mm_P2.00mm" H 5938 2550 50  0001 C CNN
+F 3 "~" H 5900 2700 50  0001 C CNN
+	1    5900 2700
+	0    1    1    0
+$EndComp
+Wire Wire Line
+	5750 2700 5600 2700
 $EndSCHEMATC
