File: Feuille2.sch (KiCad schematic (older format))
At the start: 26 parts, among them J15 Screw_Terminal_01x02, Q2 BC548, U1 LM311, U4 TL074, U5 L78L05_TO92, U6 LMC7660, U8 LM386

Commit message: V4.0-a
Parts:
- added D2: LED, LED_THT:LED_D3.0mm, symbol Device:LED
- added J14: Conn_01x02, Connector_PinHeader_2.54mm:PinHeader_1x02_P2.54mm_Vertical, symbol Connector_Generic:Conn_01x02
- added Q1: BC548, Package_TO_SOT_THT:TO-92_Inline_Wide, symbol Transistor_BJT:BC548
- added R14: 100k, Resistor_THT:R_Axial_DIN0204_L3.6mm_D1.6mm_P2.54mm_Vertical, symbol Device:R
- added R15: 100k, Resistor_THT:R_Axial_DIN0207_L6.3mm_D2.5mm_P7.62mm_Horizontal, symbol Device:R
- added R5: 10k, Resistor_THT:R_Axial_DIN0207_L6.3mm_D2.5mm_P7.62mm_Horizontal, symbol Device:R
- added R6: 330, Resistor_THT:R_Axial_DIN0207_L6.3mm_D2.5mm_P7.62mm_Horizontal, symbol Device:R
Connections:
- net GND: now also D2.1 (K), Q1.3 (E), R14.2, R15.1
- net Squelch: now also R14.1
- new net: J14.2 (Pin_2), Q1.1 (C)
- new net: Q1.2 (B), R5.1
- new net: D2.2 (A), R6.1
- new net CMD_PTT: R15.2, R5.2, R6.2
- new net EXT_PTT: J14.1 (Pin_1)
Other:
- note added: "Circuit PTT"
- note added: "J14 : \nsans/avec PTT"
- note added: "PTT"
- note added: "entrée squelch\n0 / 12V"

Commit message: V4.1
Parts:
- R16: value 600 -> 680
Other:
- moved on the sheet: U4D
Changed lines of the file:
@@
 encoding utf-8
 Sheet 2 2
-Title "Interface Raspberry V4 - MTM800(E) MTM5x00 pour SVXLink"
-Date "20/03/2021"
-Rev "4"
+Title "Interface Raspberry V4.1 - MTM800(E) MTM5x00 pour SVXLink"
+Date "20/01/2022"
+Rev "4.1"
 Comp "F1IWQ"
 Comment1 ""
@@
 L Amplifier_Operational:TL074 U4
 U 4 1 5F420A93
-P 4650 7050
-F 0 "U4" H 4650 7417 50  0000 C CNN
-F 1 "TL074" H 4650 7326 50  0000 C CNN
-F 2 "Package_SO:SOIC-14_3.9x8.7mm_P1.27mm" H 4600 7150 50  0001 C CNN
-F 3 "http://www.ti.com/lit/ds/symlink/tl071.pdf" H 4700 7250 50  0001 C CNN
-	4    4650 7050
-	1    0    0    -1
-$EndComp
-Wire Wire Line
-	4350 7150 4200 7150
-Wire Wire Line
-	4200 7150 4200 7250
-Wire Wire Line
-	4350 6950 4200 6950
-Wire Wire Line
-	4200 6950 4200 7150
-Connection ~ 4200 7150
+P 1400 6900
+F 0 "U4" H 1400 7267 50  0000 C CNN
+F 1 "TL074" H 1400 7176 50  0000 C CNN
+F 2 "Package_SO:SOIC-14_3.9x8.7mm_P1.27mm" H 1350 7000 50  0001 C CNN
+F 3 "http://www.ti.com/lit/ds/symlink/tl071.pdf" H 1450 7100 50  0001 C CNN
+	4    1400 6900
+	1    0    0    -1
+$EndComp
+Wire Wire Line
+	1100 7000 950  7000
+Wire Wire Line
+	950  7000 950  7100
+Wire Wire Line
+	1100 6800 950  6800
+Wire Wire Line
+	950  6800 950  7000
+Connection ~ 950  7000
 $Comp
 L power:GND #PWR0110
 U 1 1 5F4278DB
-P 4200 7250
-F 0 "#PWR0110" H 4200 7000 50  0001 C CNN
-F 1 "GND" H 4205 7077 50  0000 C CNN
-F 2 "" H 4200 7250 50  0001 C CNN
-F 3 "" H 4200 7250 50  0001 C CNN
-	1    4200 7250
-	1    0    0    -1
-$EndComp
-NoConn ~ 4950 7050
+P 950 7100
+F 0 "#PWR0110" H 950 6850 50  0001 C CNN
+F 1 "GND" H 955 6927 50  0000 C CNN
+F 2 "" H 950 7100 50  0001 C CNN
+F 3 "" H 950 7100 50  0001 C CNN
+	1    950  7100
+	1    0    0    -1
+$EndComp
+NoConn ~ 1700 6900
 Text GLabel 5300 4350 0    39   Input ~ 0
 12V
@@
 AR Path="/5F6D3208/5F663E1D" Ref="R16"  Part="1"
 F 0 "R16" H 3700 5400 50  0000 C CNN
-F 1 "600" H 3700 5300 50  0000 C CNN
+F 1 "680" H 3700 5300 50  0000 C CNN
 F 2 "Resistor_THT:R_Axial_DIN0207_L6.3mm_D2.5mm_P7.62mm_Horizontal" V 3780 5300 50  0001 C CNN
 F 3 "~" H 3850 5300 50  0001 C CNN
@@
 AR Path="/5F6D3208/60597F8E" Ref="#PWR0115"  Part="1"
 F 0 "#PWR0115" H 9900 5350 50  0001 C CNN
-F 1 "GND" H 9905 5427 50  0000 C CNN
+F 1 "GND" H 9900 5450 50  0000 C CNN
 F 2 "" H 9900 5600 50  0001 C CNN
 F 3 "" H 9900 5600 50  0001 C CNN
@@
 Text Notes 8600 4250 0    47   ~ 0
 Circuit PTT
-Wire Wire Line
-	9900 5150 9900 5600
 Text Notes 7050 1050 0    35   ~ 0
 entrée squelch\n0 / 12V
@@
 	8600 4950 8650 4950
 Connection ~ 8650 4950
+Wire Wire Line
+	9900 5150 9900 5600
 $EndSCHEMATC
